Commit message: feat(kortex_description): let load_arm callers supply their own ros2_control block
Add an include_ros2_control argument, default true, to load_arm in the
Gen3 7DoF, Gen3 6DoF, and Gen3 Lite macros. When false, load_arm emits
the arm's links and joints only, so the caller can choose the
<ros2_control> block itself, for example a simulator's hardware interface
that kortex.ros2_control.xacro does not know about. This mirrors the
include_ros2_control argument robotiq_description's robotiq_gripper
macro already takes.

With the default, the generated URDF is byte-identical to before for
gen3.xacro (7DoF mock and Kortex, 6DoF Gazebo) and for load_arm on the
Gen3 Lite.

Co-Authored-By: Claude Opus 5.5 <noreply@anthropic.com>

File: kortex_description/arms/gen3/6dof/urdf/gen3_macro.xacro (robot description, xacro)
@@ -29,29 +29,34 @@
     use_external_cable:=false
     initial_positions:=${dict(joint_1=0.0,joint_2=0.0,joint_3=0.0,joint_4=0.0,joint_5=0.0,joint_6=0.0)}
-    moveit_active:=false">
-    <!-- ros2 control include -->
-    <xacro:include filename="$(find kortex_description)/arms/gen3/${dof}dof/urdf/kortex.ros2_control.xacro" />
-    <xacro:kortex_ros2_control
-      name="${prefix}KortexMultiInterfaceHardware" prefix="${prefix}"
-      use_fake_hardware="${use_fake_hardware}"
-      fake_sensor_commands="${fake_sensor_commands}"
-      sim_gazebo="${sim_gazebo}"
-      sim_isaac="${sim_isaac}"
-      isaac_joint_commands="${isaac_joint_commands}"
-      isaac_joint_states="${isaac_joint_states}"
-      tf_prefix=""
-      initial_positions="${initial_positions}"
-      robot_ip="${robot_ip}"
-      username="${username}"
-      password="${password}"
-      port="${port}"
-      port_realtime="${port_realtime}"
-      session_inactivity_timeout_ms="${session_inactivity_timeout_ms}"
-      connection_inactivity_timeout_ms="${connection_inactivity_timeout_ms}"
-      use_internal_bus_gripper_comm="${use_internal_bus_gripper_comm}"
-      gripper_max_velocity="${gripper_max_velocity}"
-      gripper_max_force="${gripper_max_force}"
-      gripper_joint_name="${gripper_joint_name}"
-      gripper="${gripper}"/>
+    moveit_active:=false
+    include_ros2_control:=true">
+    <!-- ros2 control include. Set include_ros2_control:=false to leave the
+         <ros2_control> block to the caller, for example to select a different
+         hardware interface such as a simulator. -->
+    <xacro:if value="${include_ros2_control}">
+      <xacro:include filename="$(find kortex_description)/arms/gen3/${dof}dof/urdf/kortex.ros2_control.xacro" />
+      <xacro:kortex_ros2_control
+        name="${prefix}KortexMultiInterfaceHardware" prefix="${prefix}"
+        use_fake_hardware="${use_fake_hardware}"
+        fake_sensor_commands="${fake_sensor_commands}"
+        sim_gazebo="${sim_gazebo}"
+        sim_isaac="${sim_isaac}"
+        isaac_joint_commands="${isaac_joint_commands}"
+        isaac_joint_states="${isaac_joint_states}"
+        tf_prefix=""
+        initial_positions="${initial_positions}"
+        robot_ip="${robot_ip}"
+        username="${username}"
+        password="${password}"
+        port="${port}"
+        port_realtime="${port_realtime}"
+        session_inactivity_timeout_ms="${session_inactivity_timeout_ms}"
+        connection_inactivity_timeout_ms="${connection_inactivity_timeout_ms}"
+        use_internal_bus_gripper_comm="${use_internal_bus_gripper_comm}"
+        gripper_max_velocity="${gripper_max_velocity}"
+        gripper_max_force="${gripper_max_force}"
+        gripper_joint_name="${gripper_joint_name}"
+        gripper="${gripper}"/>
+    </xacro:if>
     <joint name="${prefix}base_joint" type="fixed">
       <xacro:insert_block name="origin" />

File: kortex_description/arms/gen3/7dof/urdf/gen3_macro.xacro (robot description, xacro)
@@ -29,29 +29,34 @@
     use_external_cable:=false
     initial_positions:=${dict(joint_1=0.0,joint_2=0.0,joint_3=0.0,joint_4=0.0,joint_5=0.0,joint_6=0.0,joint_7=0.0)}
-    moveit_active:=false">
-    <!-- ros2 control include -->
-    <xacro:include filename="$(find kortex_description)/arms/gen3/${dof}dof/urdf/kortex.ros2_control.xacro" />
-    <xacro:kortex_ros2_control
-      name="${prefix}KortexMultiInterfaceHardware" prefix="${prefix}"
-      use_fake_hardware="${use_fake_hardware}"
-      fake_sensor_commands="${fake_sensor_commands}"
-      sim_gazebo="${sim_gazebo}"
-      sim_isaac="${sim_isaac}"
-      isaac_joint_commands="${isaac_joint_commands}"
-      isaac_joint_states="${isaac_joint_states}"
-      tf_prefix=""
-      initial_positions="${initial_positions}"
-      robot_ip="${robot_ip}"
-      username="${username}"
-      password="${password}"
-      port="${port}"
-      port_realtime="${port_realtime}"
-      session_inactivity_timeout_ms="${session_inactivity_timeout_ms}"
-      connection_inactivity_timeout_ms="${connection_inactivity_timeout_ms}"
-      use_internal_bus_gripper_comm="${use_internal_bus_gripper_comm}"
-      gripper_max_velocity="${gripper_max_velocity}"
-      gripper_max_force="${gripper_max_force}"
-      gripper_joint_name="${gripper_joint_name}"
-      gripper="${gripper}"/>
+    moveit_active:=false
+    include_ros2_control:=true">
+    <!-- ros2 control include. Set include_ros2_control:=false to leave the
+         <ros2_control> block to the caller, for example to select a different
+         hardware interface such as a simulator. -->
+    <xacro:if value="${include_ros2_control}">
+      <xacro:include filename="$(find kortex_description)/arms/gen3/${dof}dof/urdf/kortex.ros2_control.xacro" />
+      <xacro:kortex_ros2_control
+        name="${prefix}KortexMultiInterfaceHardware" prefix="${prefix}"
+        use_fake_hardware="${use_fake_hardware}"
+        fake_sensor_commands="${fake_sensor_commands}"
+        sim_gazebo="${sim_gazebo}"
+        sim_isaac="${sim_isaac}"
+        isaac_joint_commands="${isaac_joint_commands}"
+        isaac_joint_states="${isaac_joint_states}"
+        tf_prefix=""
+        initial_positions="${initial_positions}"
+        robot_ip="${robot_ip}"
+        username="${username}"
+        password="${password}"
+        port="${port}"
+        port_realtime="${port_realtime}"
+        session_inactivity_timeout_ms="${session_inactivity_timeout_ms}"
+        connection_inactivity_timeout_ms="${connection_inactivity_timeout_ms}"
+        use_internal_bus_gripper_comm="${use_internal_bus_gripper_comm}"
+        gripper_max_velocity="${gripper_max_velocity}"
+        gripper_max_force="${gripper_max_force}"
+        gripper_joint_name="${gripper_joint_name}"
+        gripper="${gripper}"/>
+    </xacro:if>
     <joint name="${prefix}base_joint" type="fixed">
       <xacro:insert_block name="origin" />

File: kortex_description/arms/gen3_lite/6dof/urdf/gen3_lite_macro.xacro (robot description, xacro)
@@ -28,47 +28,52 @@
     use_external_cable:=false
     initial_positions:=${dict(joint_1=0.0,joint_2=0.0,joint_3=0.0,joint_4=0.0,joint_5=0.0,joint_6=0.0)}
-    moveit_active:=false" >
-    <!-- ros2 control include -->
-    <xacro:include filename="$(find kortex_description)/arms/gen3_lite/${dof}dof/urdf/kortex.ros2_control.xacro" />
-    <xacro:if value="${sim_gazebo}">
-      <xacro:unless value="${moveit_active}">
-        <xacro:property name="ros2_control_name" value="GazeboSimSystem"/>
+    moveit_active:=false
+    include_ros2_control:=true" >
+    <!-- ros2 control include. Set include_ros2_control:=false to leave the
+         <ros2_control> block to the caller, for example to select a different
+         hardware interface such as a simulator. -->
+    <xacro:if value="${include_ros2_control}">
+      <xacro:include filename="$(find kortex_description)/arms/gen3_lite/${dof}dof/urdf/kortex.ros2_control.xacro" />
+      <xacro:if value="${sim_gazebo}">
+        <xacro:unless value="${moveit_active}">
+          <xacro:property name="ros2_control_name" value="GazeboSimSystem"/>
+        </xacro:unless>
+      </xacro:if>
+       <xacro:if value="${use_fake_hardware}">
+        <xacro:unless value="${moveit_active}">
+          <xacro:property name="ros2_control_name" value="GenericSystem"/>
+        </xacro:unless>
+      </xacro:if>
+      <xacro:unless value="${use_fake_hardware or sim_gazebo}">
+        <xacro:unless value="${moveit_active}">
+          <xacro:property name="ros2_control_name" value="${prefix}KortexMultiInterfaceHardware"/>
+        </xacro:unless>
       </xacro:unless>
+      <xacro:if value="${moveit_active}">
+        <xacro:property name="ros2_control_name" value="${prefix}KortexMultiInterfaceHardware"/>
+      </xacro:if>
+      <xacro:kortex_ros2_control
+        name="${ros2_control_name}" prefix="${prefix}"
+        use_fake_hardware="${use_fake_hardware}"
+        fake_sensor_commands="${fake_sensor_commands}"
+        sim_gazebo="${sim_gazebo}"
+        sim_isaac="${sim_isaac}"
+        isaac_joint_commands="${isaac_joint_commands}"
+        isaac_joint_states="${isaac_joint_states}"
+        tf_prefix=""
+        initial_positions="${initial_positions}"
+        robot_ip="${robot_ip}"
+        username="${username}"
+        password="${password}"
+        port="${port}"
+        port_realtime="${port_realtime}"
+        session_inactivity_timeout_ms="${session_inactivity_timeout_ms}"
+        connection_inactivity_timeout_ms="${connection_inactivity_timeout_ms}"
+        use_internal_bus_gripper_comm="${use_internal_bus_gripper_comm}"
+        gripper_max_velocity="${gripper_max_velocity}"
+        gripper_max_force="${gripper_max_force}"
+        gripper_joint_name="${gripper_joint_name}"
+        moveit_active="${moveit_active}"/>
     </xacro:if>
-     <xacro:if value="${use_fake_hardware}">
-      <xacro:unless value="${moveit_active}">
-        <xacro:property name="ros2_control_name" value="GenericSystem"/>
-      </xacro:unless>
-    </xacro:if>
-    <xacro:unless value="${use_fake_hardware or sim_gazebo}">
-      <xacro:unless value="${moveit_active}">
-        <xacro:property name="ros2_control_name" value="${prefix}KortexMultiInterfaceHardware"/>
-      </xacro:unless>
-    </xacro:unless>
-    <xacro:if value="${moveit_active}">
-      <xacro:property name="ros2_control_name" value="${prefix}KortexMultiInterfaceHardware"/>
-    </xacro:if>
-    <xacro:kortex_ros2_control
-      name="${ros2_control_name}" prefix="${prefix}"
-      use_fake_hardware="${use_fake_hardware}"
-      fake_sensor_commands="${fake_sensor_commands}"
-      sim_gazebo="${sim_gazebo}"
-      sim_isaac="${sim_isaac}"
-      isaac_joint_commands="${isaac_joint_commands}"
-      isaac_joint_states="${isaac_joint_states}"
-      tf_prefix=""
-      initial_positions="${initial_positions}"
-      robot_ip="${robot_ip}"
-      username="${username}"
-      password="${password}"
-      port="${port}"
-      port_realtime="${port_realtime}"
-      session_inactivity_timeout_ms="${session_inactivity_timeout_ms}"
-      connection_inactivity_timeout_ms="${connection_inactivity_timeout_ms}"
-      use_internal_bus_gripper_comm="${use_internal_bus_gripper_comm}"
-      gripper_max_velocity="${gripper_max_velocity}"
-      gripper_max_force="${gripper_max_force}"
-      gripper_joint_name="${gripper_joint_name}"
-      moveit_active="${moveit_active}"/>
     <joint name="${prefix}base_joint" type="fixed">
       <xacro:insert_block name="origin" />
